Commit message: first commit

File: orne_box_description/urdf/links/base_link.urdf.xacro (robot description, xacro)
@@ -2,4 +2,12 @@
 <robot xmlns:xacro="http://www.ros.org/wiki/xacro">
   <xacro:macro name="base_link">
+    <!-- base_footprint-->
+    <link name="base_footprint"/>
+    <joint name="base_joint" type="fixed">
+      <origin xyz="0.0 0.0 0.0"/>
+      <parent link="base_footprint"/>
+      <child link="base_link"/>
+    </joint>
+    <!-- base_link -->
     <link name="base_link">
       <visual>

File: orne_box_description/urdf/orne_box.gazebo.xacro (robot description, xacro)
@@ -4,5 +4,4 @@
   <xacro:arg name="laser_visual" default="true"/>
   <xacro:arg name="imu_visual" default="false"/>
-  <xacro:arg name="ignition_gazebo" default="false"/>
   <xacro:arg name="enable_camera" default="false"/>
   <gazebo reference="left_caster_wheel_link">
@@ -41,9 +40,34 @@
   </gazebo>
   <!-- @TODO More clear boolean operation -->
-  <xacro:if value="${'$(arg ignition_gazebo)' == 'false'}">
-    <gazebo>
+    <!-- <gazebo>
       <plugin name="gazebo_ros_control" filename="libgazebo_ros_control.so">
         <robotNamespace>orne_box</robotNamespace>
         <robotSimType>gazebo_ros_control/DefaultRobotHWSim</robotSimType>
+      </plugin>
+    </gazebo> -->
+    <gazebo>
+      <plugin name="gazebo_ros_control" filename="libgazebo_ros_diff_drive.so">
+        <always_on>true</always_on>
+        <robotNamespace>/orne_box</robotNamespace>
+        <!-- frame and cmd_vel -->
+        <command_topic>cmd_vel</command_topic>
+        <odometry_topic>odom</odometry_topic>
+        <odometry_frame>odom</odometry_frame>
+        <!-- <odometrySource>world</odometrySource> -->
+        <robot_base_frame>base_footprint</robot_base_frame>
+        <update_rate>30</update_rate>
+        <!-- wheels -->
+        <left_joint>left_wheel_joint</left_joint>
+        <right_joint>right_wheel_joint</right_joint>
+        <!-- kinematics -->
+        <wheel_separation>0.46</wheel_separation>
+        <wheel_diameter>0.304</wheel_diameter>
+        <wheel_acceleration>1</wheel_acceleration>
+        <max_wheel_torque>20</max_wheel_torque>
+        <max_wheel_acceleration>1.0</max_wheel_acceleration>
+        <!-- output -->
+        <publish_odom>true</publish_odom>
+        <publish_odom_tf>true</publish_odom_tf>
+        <publish_wheel_tf>false</publish_wheel_tf>
       </plugin>
     </gazebo>
@@ -51,8 +75,70 @@
       <material>Gazebo/Orange</material>
     </gazebo>
+    <!-- imu -->
     <gazebo reference="imu_link">
       <sensor type="imu" name="imu">
+        <plugin filename="libgazebo_ros_imu_sensor.so" name="imu_plugin">
+          <ros>
+            <remapping>~/out:=imu</remapping>
+          </ros>
+          <initial_orientation_as_reference>false</initial_orientation_as_reference>
+        </plugin>
         <always_on>true</always_on>
-        <visualize>$(arg imu_visual)</visualize>
+        <update_rate>100</update_rate>
+        <visualize>true</visualize>
+        <imu>
+        <angular_velocity>
+          <x>
+            <noise type="gaussian">
+                <mean>0.0</mean>
+                <stddev>2e-4</stddev>
+                <bias_mean>0.0000075</bias_mean>
+                <bias_stddev>0.0000008</bias_stddev>
+              </noise>
+            </x>
+            <y>
+              <noise type="gaussian">
+                <mean>0.0</mean>
+                <stddev>2e-4</stddev>
+                <bias_mean>0.0000075</bias_mean>
+                <bias_stddev>0.0000008</bias_stddev>
+              </noise>
+            </y>
+            <z>
+              <noise type="gaussian">
+                <mean>0.0</mean>
+                <stddev>2e-4</stddev>
+                <bias_mean>0.0000075</bias_mean>
+                <bias_stddev>0.0000008</bias_stddev>
+              </noise>
+            </z>
+          </angular_velocity>
+          <linear_acceleration>
+            <x>
+              <noise type="gaussian">
+                <mean>0.0</mean>
+                <stddev>1.7e-2</stddev>
+                <bias_mean>0.1</bias_mean>
+                <bias_stddev>0.001</bias_stddev>
+              </noise>
+            </x>
+            <y>
+              <noise type="gaussian">
+                <mean>0.0</mean>
+                <stddev>1.7e-2</stddev>
+                <bias_mean>0.1</bias_mean>
+                <bias_stddev>0.001</bias_stddev>
+              </noise>
+            </y>
+            <z>
+              <noise type="gaussian">
+                <mean>0.0</mean>
+                <stddev>1.7e-2</stddev>
+                <bias_mean>0.1</bias_mean>
+                <bias_stddev>0.001</bias_stddev>
+              </noise>
+            </z>
+          </linear_acceleration>
+        </imu>
       </sensor>
       <material>Gazebo/Green</material>
@@ -92,201 +178,13 @@
           </noise>
         </ray>
-        <plugin name="gazebo_ros_head_hokuyo_controller" filename="libgazebo_ros_laser.so">
-          <topicName>/scan</topicName>
-          <frameName>hokuyo_link</frameName>
+        <plugin name="gazebo_ros_head_hokuyo_controller" filename="libgazebo_ros_ray_sensor.so">
+          <ros>
+            <remapping>~/out:=scan</remapping>
+          </ros>
+          <frame_name>hokuyo_link</frame_name>
+          <output_type>sensor_msgs/LaserScan</output_type>
         </plugin>
       </sensor>
       <material>Gazebo/Black</material>
     </gazebo>
-  </xacro:if>
-  <xacro:if value="$(arg ignition_gazebo)">
-    <gazebo>
-      <static>false</static>
-      <selfCollide>true</selfCollide>
-      <plugin filename="ignition-gazebo-joint-state-publisher-system" name="ignition::gazebo::systems::JointStatePublisher">
-        <topic>model/orne_box/joint_states</topic>
-      </plugin>
-      <plugin filename="ignition-gazebo-pose-publisher-system" name="ignition::gazebo::systems::PosePublisher">
-        <publish_link_pose>true</publish_link_pose>
-        <publish_collision_pose>true</publish_collision_pose>
-        <publish_visual_pose>false</publish_visual_pose>
-        <publish_nested_model_pose>false</publish_nested_model_pose>
-      </plugin>
-      <plugin filename="ignition-gazebo-diff-drive-system" name="ignition::gazebo::systems::DiffDrive">
-        <left_joint>left_wheel_joint</left_joint>
-        <right_joint>right_wheel_joint</right_joint>
-        <wheel_separation>0.38</wheel_separation>
-        <wheel_radius>0.152</wheel_radius>
-        <odom_publish_frequency>30</odom_publish_frequency>
-        <max_angular_acceleration>3.14</max_angular_acceleration>
-        <min_angular_acceleration>-3.14</min_angular_acceleration>
-        <max_angular_velocity>1.57</max_angular_velocity>
-        <min_angular_velocity>-1.57</min_angular_velocity>
-      </plugin>
-      <plugin filename="libignition-gazebo-wheel-slip-system.so" name="ignition::gazebo::systems::WheelSlip">
-        <wheel link_name="left_caster_wheel_link">
-          <slip_compliance_lateral>0.2</slip_compliance_lateral>
-          <slip_compliance_longitudinal>0.15</slip_compliance_longitudinal>
-          <wheel_normal_force>20.6</wheel_normal_force>
-          <wheel_radius>0.04</wheel_radius>
-        </wheel>
-        <wheel link_name="right_caster_wheel_link">
-          <slip_compliance_lateral>0.2</slip_compliance_lateral>
-          <slip_compliance_longitudinal>0.15</slip_compliance_longitudinal>
-          <wheel_normal_force>20.6</wheel_normal_force>
-          <wheel_radius>0.04</wheel_radius>
-        </wheel>
-        <wheel link_name="wheel_left_link">
-          <slip_compliance_lateral>0.7</slip_compliance_lateral>
-          <slip_compliance_longitudinal>0.55</slip_compliance_longitudinal>
-          <wheel_normal_force>294.6</wheel_normal_force>
-          <wheel_radius>0.15</wheel_radius>
-        </wheel>
-        <wheel link_name="wheel_right_link">
-          <slip_compliance_lateral>0.7</slip_compliance_lateral>
-          <slip_compliance_longitudinal>0.55</slip_compliance_longitudinal>
-          <wheel_normal_force>294.6</wheel_normal_force>
-          <wheel_radius>0.15</wheel_radius>
-        </wheel>
-      </plugin>
-    </gazebo>
-    <gazebo reference="hokuyo_link">
-      <sensor type="gpu_lidar" name="head_hokuyo_sensor">
-        <pose>0 0 0 0 0 0</pose>
-        <visualize>$(arg laser_visual)</visualize>
-        <update_rate>40</update_rate>
-        <topic>model/orne_box/hokuyo_scan</topic>
-        <lidar>
-          <scan>
-            <horizontal>
-              <samples>361</samples>
-              <resolution>1</resolution>
-              <min_angle>${-PI/180*110}</min_angle>
-              <max_angle>${ PI/180*110}</max_angle>
-            </horizontal>
-            <vertical>
-              <samples>1</samples>
-              <resolution>1</resolution>
-            </vertical>
-          </scan>
-          <range>
-            <min>0.10</min>
-            <max>30.0</max>
-            <resolution>0.01</resolution>
-          </range>
-          <noise>
-            <type>gaussian</type>
-            <mean>0.0</mean>
-            <stddev>0.01</stddev>
-          </noise>
-        </lidar>
-      </sensor>
-    </gazebo>
-    <gazebo reference="imu_link">
-      <sensor name="imu_link" type="imu">
-        <always_on>1</always_on>
-        <update_rate>200</update_rate>
-        <visualize>false</visualize>
-        <topic>model/orne_box/imu</topic>
-        <imu>
-          <angular_velocity>
-            <x>
-              <noise type="gaussian">
-                <mean>0.0</mean>
-                <stddev>0.1</stddev>
-              </noise>
-            </x>
-            <y>
-              <noise type="gaussian">
-                <mean>0.0</mean>
-                <stddev>0.1</stddev>
-              </noise>
-            </y>
-            <z>
-              <noise type="gaussian">
-                <mean>0.0</mean>
-                <stddev>0.2</stddev>
-              </noise>
-            </z>
-          </angular_velocity>
-          <linear_acceleration>
-            <x>
-              <noise type="gaussian">
-                <mean>0.0</mean>
-                <stddev>0.1</stddev>
-              </noise>
-            </x>
-            <y>
-              <noise type="gaussian">
-                <mean>0.0</mean>
-                <stddev>0.1</stddev>
-              </noise>
-            </y>
-            <z>
-              <noise type="gaussian">
-                <mean>0.0</mean>
-                <stddev>0.2</stddev>
-              </noise>
-            </z>
-          </linear_acceleration>
-        </imu>
-      </sensor>
-    </gazebo>
-    <xacro:if value="$(arg enable_camera)">
-      <gazebo reference="zed_camera_center">
-        <sensor name="zed_camera_center" type="camera">
-          <always_on>1</always_on>
-          <update_rate>15</update_rate>
-          <visualize>false</visualize>
-          <topic>model/orne_box/zed_node/image</topic>
-          <camera>
-            <horizontal_fov>1.919805</horizontal_fov>
-            <image>
-              <width>1920</width>
-              <height>1080</height>
-            </image>
-            <clip>
-              <near>0.01</near>
-              <far>50</far>
-            </clip>
-            <noise>
-              <type>gaussian</type>
-              <mean>0.0</mean>
-              <stddev>0.025</stddev>
-            </noise>
-          </camera>
-        </sensor>
-        <sensor name="zed_depth_camera_center" type="depth_camera">
-          <pose>0 0 -0.8 3.14 -0.38 0</pose>
-          <always_on>1</always_on>
-          <update_rate>15</update_rate>
-          <visualize>false</visualize>
-          <topic>model/orne_box/zed_node/depth_image</topic>
-          <camera>
-            <horizontal_fov>1.919805</horizontal_fov>
-            <image>
-              <width>1280</width>
-              <height>720</height>
-            </image>
-            <clip>
-              <near>0.4</near>
-              <far>6</far>
-            </clip>
-            <noise>
-              <type>gaussian</type>
-              <mean>0.0</mean>
-              <stddev>0.1</stddev>
-            </noise>
-          </camera>
-        </sensor>
-      </gazebo>
-    </xacro:if>
-    <gazebo reference="gnss_link">
-      <sensor name="gnss_link" type="navsat">
-        <always_on>1</always_on>
-        <update_rate>1</update_rate>
-        <topic>model/orne_box/navsat</topic>
-      </sensor>
-    </gazebo>
-  </xacro:if>
 </robot>

File: orne_box_description/urdf/orne_box.urdf.xacro (robot description, xacro)
@@ -11,5 +11,5 @@
   <xacro:include filename="$(find orne_box_description)/urdf/joints/caster_swivel_joint.urdf.xacro"/>
   <xacro:include filename="$(find orne_box_description)/urdf/joints/wheel_joint.urdf.xacro"/>
-  <!-- <xacro:include filename="$(find orne_box_description)/urdf/sensors/imu.urdf.xacro"/> -->
+  <xacro:include filename="$(find orne_box_description)/urdf/sensors/imu.urdf.xacro"/>
   <xacro:include filename="$(find orne_box_description)/urdf/sensors/hokuyo.urdf.xacro"/>
   <!-- Setting for base -->
@@ -48,12 +48,14 @@
     <origin xyz="0.23 0.0 0.270" rpy="${-PI} 0 ${PI/2}"/>
   </xacro:sensor_imu> -->
+  <xacro:sensor_imu name="imu" parent="base_link" size="0.05 0.05 0.05">
+    <origin xyz="0.23 0.0 0.270" rpy="0 0 0"/>
+    <origin_child xyz="0.0 0.0 0.0" rpy="0 0 0"/>
+  </xacro:sensor_imu>
   <!-- Setting for 2D-LiDAR -->
   <xacro:sensor_hokuyo name="hokuyo" parent="base_link" size="0.05 0.05 0.05">
-    <!--origin xyz="0.374295 0 0.2185" rpy="${-PI} 0 0"/-->
-    <!-- <origin xyz="0.23 0 0.4" rpy="0 0 0"/> -->
-    <origin xyz="0.34 0 0.21" rpy="0 0 0"/>
+    <origin xyz="0.374295 0 0.2185" rpy="${-PI} 0 0"/>
   </xacro:sensor_hokuyo>
-  <!-- <xacro:sensor_hokuyo name="mirror_lidar" parent="base_link" size="0.05 0.05 0.05">
-    <origin xyz="-0.08 0.0 0.7" rpy="${-PI} 0.175 0"/>
-  </xacro:sensor_hokuyo> -->
+  <xacro:sensor_hokuyo name="mirror_lidar" parent="base_link" size="0.05 0.05 0.05">
+    <origin xyz="0.43 0.0 0.34" rpy="0 0.314 0"/>
+  </xacro:sensor_hokuyo>
 </robot>

File: orne_box_description/urdf/orne_box_3d_lidar.urdf.xacro (robot description, xacro)
@@ -73,11 +73,9 @@
     </gazebo>
   </xacro:if>
-  <xacro:include filename="$(find orne_box_description)/urdf/sensors/gnss.urdf.xacro"/>
+  <xacro:include filename="$(find orne_box_description)/urdf/sensors/gnss.urdf.xacro"/> -->
   <xacro:include filename="$(find orne_box_description)/urdf/sensors/camera.urdf.xacro"/>
-  <!-- Setting for GNSS -->
   <xacro:sensor_gnss name="gnss" parent="base_link">
     <origin xyz="-0.12 0.12 0.9" rpy="0 0 0"/>
   </xacro:sensor_gnss>
-  <!-- Setting for Camera -->
   <xacro:sensor_camera name="camera" parent="base_link">
     <origin xyz="-0.08 0.0 0.8" rpy="0 0.38 0"/>

File: orne_box_description/urdf/sensors/imu.urdf.xacro (robot description, xacro)
@@ -1,6 +1,5 @@
 <?xml version="1.0"?>
 <robot xmlns:xacro="http://ros.org/wiki/xacro" xmlns:controller="http://playerstage.sourceforge.net/gazebo/xmlschema/#controller" xmlns:interface="http://playerstage.sourceforge.net/gazebo/xmlschema/#interface" name="sensor_imu">
-  <xacro:arg name="ignition_gazebo" default="false"/>
-  <xacro:macro name="sensor_imu" params="name parent *origin size">
+  <xacro:macro name="sensor_imu" params="name parent *origin *origin_child size">
     <joint name="${name}_joint" type="fixed">
       <axis xyz="1 0 0"/>
@@ -9,5 +8,26 @@
       <child link="${name}_link"/>
     </joint>
+    <!-- <link name="${name}_link"> -->
     <link name="${name}_link">
+      <inertial>
+        <origin xyz="0.0 0.0 0.0" rpy="0.0 0.0 0.0"/>
+        <mass value="0.005"/>
+        <inertia ixx="0.001" ixy="0.0" ixz="0.0" iyy="0.001" iyz="0.0" izz="0.001"/>
+      </inertial>
+      <visual>
+        <!-- <origin rpy="0 0 0" xyz="0 0 0"/>
+        <geometry>
+          <box size="${size}"/>
+        </geometry>
+        <material name="green"/> -->
+      </visual>
+    </link>
+    <joint name="${name}_base_joint" type="fixed">
+      <axis xyz="1 0 0"/>
+      <xacro:insert_block name="origin_child"/>
+      <parent link="${name}_link"/>
+      <child link="${name}"/>
+    </joint>
+    <link name="${name}">
       <inertial>
         <origin xyz="0.0 0.0 0.0" rpy="0.0 0.0 0.0"/>
@@ -23,16 +43,4 @@
       </visual>
     </link>
-    <xacro:if value="${'$(arg ignition_gazebo)' == 'false'}">
-      <gazebo>
-        <plugin name="ros_imu" filename="libgazebo_ros_imu.so">
-          <bodyName>${parent}</bodyName> <!-- bodyName always set base_link by URDF parser -->
-          <topicName>imu_data</topicName>
-          <serviceName>imu_service</serviceName>
-          <gaussianNoise>0.005</gaussianNoise>
-          <updateRate>100.0</updateRate>
-          <frameName>${parent}</frameName>
-        </plugin>
-      </gazebo>
-    </xacro:if>
   </xacro:macro>
 </robot>
