Commit message: IMUを削除し2DLiDARの位置を変更

File: orne_box_description/urdf/orne_box.urdf.xacro (robot description, xacro)
@@ -45,11 +45,12 @@
   </xacro:wheel_link>
   <!-- Setting for IMU -->
-  <xacro:sensor_imu name="imu" parent="base_link" size="0.05 0.05 0.05">
+  <!-- <xacro:sensor_imu name="imu" parent="base_link" size="0.05 0.05 0.05">
     <origin xyz="0.23 0.0 0.270" rpy="${-PI} 0 ${PI/2}"/>
-  </xacro:sensor_imu>
+  </xacro:sensor_imu> -->
   <!-- Setting for 2D-LiDAR -->
   <xacro:sensor_hokuyo name="hokuyo" parent="base_link" size="0.05 0.05 0.05">
     <!--origin xyz="0.374295 0 0.2185" rpy="${-PI} 0 0"/-->
-    <origin xyz="0.23 0 0.4" rpy="0 0 0"/>
+    <!-- <origin xyz="0.23 0 0.4" rpy="0 0 0"/> -->
+    <origin xyz="0.36 0 0.19" rpy="0 0 0"/>
   </xacro:sensor_hokuyo>
   <!-- <xacro:sensor_hokuyo name="mirror_lidar" parent="base_link" size="0.05 0.05 0.05">

Commit message: update urdf

File: orne_box_description/urdf/orne_box.urdf.xacro (robot description, xacro)
@@ -52,5 +52,5 @@
     <!--origin xyz="0.374295 0 0.2185" rpy="${-PI} 0 0"/-->
     <!-- <origin xyz="0.23 0 0.4" rpy="0 0 0"/> -->
-    <origin xyz="0.36 0 0.19" rpy="0 0 0"/>
+    <origin xyz="0.335 0 0.22" rpy="0 0 0"/>
   </xacro:sensor_hokuyo>
   <!-- <xacro:sensor_hokuyo name="mirror_lidar" parent="base_link" size="0.05 0.05 0.05">

Commit message: 2DLiDARを腰の位置に設定

File: orne_box_description/urdf/orne_box.urdf.xacro (robot description, xacro)
@@ -52,5 +52,5 @@
     <!--origin xyz="0.374295 0 0.2185" rpy="${-PI} 0 0"/-->
     <!-- <origin xyz="0.23 0 0.4" rpy="0 0 0"/> -->
-    <origin xyz="0.335 0 0.22" rpy="0 0 0"/>
+    <origin xyz="-0.08 0 0.775" rpy="0 0 0"/>
   </xacro:sensor_hokuyo>
   <!-- <xacro:sensor_hokuyo name="mirror_lidar" parent="base_link" size="0.05 0.05 0.05">

Commit message: 2DLiDARの位置をロボットの下に設定

File: orne_box_description/urdf/orne_box.urdf.xacro (robot description, xacro)
@@ -52,5 +52,5 @@
     <!--origin xyz="0.374295 0 0.2185" rpy="${-PI} 0 0"/-->
     <!-- <origin xyz="0.23 0 0.4" rpy="0 0 0"/> -->
-    <origin xyz="-0.08 0 0.775" rpy="0 0 0"/>
+    <origin xyz="0.34 0 0.21" rpy="0 0 0"/>
   </xacro:sensor_hokuyo>
   <!-- <xacro:sensor_hokuyo name="mirror_lidar" parent="base_link" size="0.05 0.05 0.05">

Commit message: 津田沼チャレンジ2024年2月

File: orne_box_description/urdf/orne_box.urdf.xacro (robot description, xacro)
@@ -49,11 +49,11 @@
   </xacro:sensor_imu> -->
   <xacro:sensor_imu name="imu" parent="base_link" size="0.05 0.05 0.05">
-    <origin xyz="0.23 0.0 0.270" rpy="0 0 0"/>
+    <origin xyz="-0.04 0.0 0.28" rpy="0 0 0"/>
     <origin_child xyz="0.0 0.0 0.0" rpy="0 0 0"/>
   </xacro:sensor_imu>
   <!-- Setting for 2D-LiDAR -->
-  <xacro:sensor_hokuyo name="hokuyo" parent="base_link" size="0.05 0.05 0.05">
+  <!-- <xacro:sensor_hokuyo name="hokuyo" parent="base_link" size="0.05 0.05 0.05">
     <origin xyz="0.374295 0 0.2185" rpy="${-PI} 0 0"/>
-  </xacro:sensor_hokuyo>
+  </xacro:sensor_hokuyo> -->
   <xacro:sensor_hokuyo name="mirror_lidar" parent="base_link" size="0.05 0.05 0.05">
     <origin xyz="0.43 0.0 0.34" rpy="0 0.314 0"/>

File: orne_box_description/urdf/orne_box_3d_lidar.urdf.xacro (robot description, xacro)
@@ -8,5 +8,6 @@
     <!-- Setting for 3D-LiDAR -->
     <xacro:VLP-16 parent="base_link" name="surestar" topic="/rfans_points" organize_cloud="false" hz="10" samples="440" gpu="false">
-      <origin xyz="0.23 0 0.40" rpy="0 0 0"/>
+      <!-- <origin xyz="0.23 0 0.40" rpy="0 0 0"/> -->
+      <origin xyz="-0.105 0 0.80" rpy="0 0 0"/>
     </xacro:VLP-16>
   </xacro:if>
@@ -73,5 +74,5 @@
     </gazebo>
   </xacro:if>
-  <xacro:include filename="$(find orne_box_description)/urdf/sensors/gnss.urdf.xacro"/> -->
+  <!-- <xacro:include filename="$(find orne_box_description)/urdf/sensors/gnss.urdf.xacro"/>
   <xacro:include filename="$(find orne_box_description)/urdf/sensors/camera.urdf.xacro"/>
   <xacro:sensor_gnss name="gnss" parent="base_link">
@@ -80,4 +81,4 @@
   <xacro:sensor_camera name="camera" parent="base_link">
     <origin xyz="-0.08 0.0 0.8" rpy="0 0.38 0"/>
-  </xacro:sensor_camera>
+  </xacro:sensor_camera> -->
 </robot>
